File: EE192_Sp17_Team01_combo.brd (EAGLE design)
At the start: 216.8 x 88.9 mm, 90 parts, among them J1 FRDM-K64F, Q1 IRFS3006PBF, Q2 IRFS3006PBF, Q3 IRFS3006PBF, Q4 IRFS3006PBF, Q5 IRFS3006PBF, Q6 IRFS3006PBF, Q7 IRFS3006PBF

Commit message: Add rev 2 boards
Add rev 2 boards, update to MCU and power circuitry
Parts:
- removed C7: (no value), rcl:C0805
- removed PWR_OUT: (no value), ee192TomasVersion:1X03-MTA
- removed U$1: TAMIYA, ee192TomasVersion:TAMIYA
- added C13: (no value), rcl:C0805
- added CONN1, CONN2, CONN3: ANDERSON_PP_DOUBLEVERTICAL, ee192:ANDERSON_PP_DOUB_VERT
- added LED1: (no value), led:CHIPLED_0805
- added MCU_PWR: (no value), ee192:1X03-MTA
- added MOTOR_PWR1: ANDERSON_PP_TRIPVERT, ee192:ANDERSON_PP_TRIP_VERT
- added R34, R35: 50kohm, rcl:R0805
- added SV1, SV2, SV3, SV4: (no value), con-lstb:MA08-2
- added U$5: TAMIYA, ee192:TAMIYA
- 3.3V_REGULATOR: device v-reg:TO220L1 -> v-reg:78MXXL
- D1: value BAT60J -> 1N5908; device diode:SOD323_ST -> diode:C4111-15
- MOTOR_PWR: value ANDERSON_PP_TRIPHORIZ -> ANDERSON_PP_DOUBLEVERTICAL; device ee192:ANDERSON_PP_TRIP_HORZ -> ee192:ANDERSON_PP_DOUB_VERT
- Q1, Q2, Q3, Q4, Q5, Q6: value IRFS3006PBF -> (none); device ee192TomasVersion:IRFS3006PBF -> ee192:TO263
- R1, R2: value 50ohm -> (none); device rcl:R0805 -> resistor:R0805
- R11, R7: value 10kohm -> 50ohm
- R13, R14: value 50kohm -> 10kohm
- moved R18 204.7 mm to (113.0, 199.4)
- moved R19 203.9 mm to (108.0, 210.8), turned to 180 degrees
- moved DOWN 200.4 mm to (8.13, 21.6)
- moved UP 200.3 mm to (8.13, 34.3), turned to 0 degrees
- moved SELECT 200.2 mm to (8.13, 48.0)
- moved ESTOP 196.9 mm to (10.2, 64.8)
- moved R11 182.9 mm to (73.7, 205.7), turned to 180 degrees
- moved R22 180.4 mm to (19.1, 19.3), turned to 180 degrees
- moved R23 180.4 mm to (19.1, 32.0), turned to 180 degrees
- moved R31 180.3 mm to (19.1, 45.7), turned to 180 degrees
- moved RESET 171.6 mm to (22.9, 69.8)
- moved R13 165.9 mm to (66.0, 198.1), turned to 90 degrees
- moved C4 163.2 mm to (106.7, 179.1), turned to 0 degrees
- moved SERVO 160.8 mm to (99.1, 160.0)
- moved HALL_MCU 157.2 mm to (64.8, 160.0)
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Connections:
- removed net 5V_SERVO: 3.3V_REGULATOR.3, 31.1, C26.+, C27.+, HALL_SENSOR.6, L1.P$2, PWR_OUT.1, R20.2, SERVO.2
- removed net N$35 (its old number): Q4.G, R2.2, R8.2
- removed net PTA1: J1.J1-8, UP.3
- removed net PTA2: DOWN.3, J1.J1-12
- removed net PTB9: J1.J1-6, SELECT.3
- new net 3V3: 3.3V_REGULATOR.OUT, 32.1, MCU_PWR.1
- new net CONN_15_16: SV4.16, SV4.2
- new net DOWN: DOWN.3, J1.J2-10
- new net HA_OUT: J1.J4-8, R1.2, R2.2
- new net N$13: SV2.10, SV2.12, SV2.14, SV2.16, SV2.2, SV2.4, SV2.6, SV2.8
- new net N$38: Q6.1, R4.2, R8.1
- new net N$39: Q2.1, R6.2, R9.2
- new net N$46: Q4.1, R14.2, R3.2
- new net N$47: Q5.1, R10.1, R7.2
- new net N$52: Q1.1, R11.2, R12.1
- new net N$53: LED1.C, MOTOR_PREDRIVER.22
- new net N$54: LED1.A, R15.2
- new net N$6: SV3.16, SV3.2
- new net N$7: SV3.1, SV3.15
- new net RST_SCRN: J1.J2-8, SCREEN.3
- new net SELECT: J1.J2-4, SELECT.3
- new net UP: J1.J2-6, UP.3
- net 3.3V: now also CAMERA1.2, CAMERA2.2
- net 5V: now also SCREEN.4; no longer CAMERA1.2, CAMERA2.2, SCREEN.1
- net BRAKEN: now also J1.J1-6, R18.1; no longer J1.J2-10, R16.1
- net CELL_A: now also BATT_SENSE.3; no longer BATT_SENSE.2
- net CELL_AB: now also BATT_SENSE.2; no longer BATT_SENSE.3
- net CELL_ABC: now also BATT_SENSE.1; no longer BATT_SENSE.4
- net CLK: now also SCREEN.2; no longer SCREEN.5
- net CLK_CAM1: now also CAMERA1.3; no longer CAMERA1.4
- net CLK_CAM2: now also CAMERA2.3; no longer CAMERA2.4
- net DATA: now also SCREEN.1; no longer SCREEN.4
- net DIR: now also R17.1; no longer R14.1
- net ENABLE: now also R16.1; no longer R13.1
- net GHA: now also R4.1; no longer R1.1
- net GHB: now also R3.1; no longer R2.1
- net GHC: now also R6.1; no longer R3.1
- net GLA: now also R7.1; no longer R4.1
- net GLC: now also R11.1; no longer R6.1
- net GND: now also 3.3V_REGULATOR.GND, BATT_SENSE.4, C13.2, CONN1.PIN1, CONN2.PIN1, CONN3.PIN1, MCU_PWR.3, MOTOR_PWR.PIN1, Q1.2, Q3.2, Q5.2, R17.2, R18.2, R2.1, SCREEN.5, U$5.-; no longer 3.3V_REGULATOR.1, BATT_SENSE.1, C7.2, PWR_OUT.3, Q1.S, Q3.S, Q5.S, R11.2, R14.2, SCREEN.2, U$1.-
- net HA: now also HALL_MCU.3, R1.1, R35.2; no longer HALL_MCU.1, J1.J2-6, R19.2
- net HB: now also J1.J1-12, R34.2; no longer R18.2
- net HC: now also HALL_MCU.1, R19.2; no longer HALL_MCU.3, R17.2
- net MEAS_CELL_A: now also BATT_SENSE1.4; no longer BATT_SENSE1.2, BMS.4
- net MEAS_CELL_C: now also BATT_SENSE1.2, BMS.4; no longer BATT_SENSE1.4
- net N$10: now also SV3.14; no longer Q1.G, R12.1, R6.2
- net N$2: now also SV2.1, SV2.11, SV2.13, SV2.15, SV2.3, SV2.5, SV2.7, SV2.9; no longer Q3.G, R11.1, R5.2
- net N$22: now also SV1.10, SV1.12, SV1.14, SV1.16, SV1.2, SV1.4, SV1.6, SV1.8; no longer Q6.G, R1.2, R7.1
- net N$26: now also SV1.1, SV1.11, SV1.13, SV1.15, SV1.3, SV1.5, SV1.7, SV1.9; no longer Q5.G, R10.1, R4.2
- net N$32: now also SV4.1, SV4.15; no longer Q2.G, R3.2, R9.2
- net N$40: now also Q3.1, R13.1, R5.2; no longer J1.J4-8
- net N$5: no longer MOTOR_PREDRIVER.22, R15.2
- net PWM_SERVO: now also J1.J1-8; no longer J1.J2-8
- net RST: no longer J1.J2-4, SCREEN.3
- net SA: now also C13.1, MOTOR_PWR1.PIN3, Q5.3, Q6.2, R8.2; no longer C7.1, MOTOR_PWR.PIN3, MOTOR_PWR.PIN3-LEAD, Q5.D, Q6.S, R7.2
- net SB: now also MOTOR_PWR1.PIN2, Q3.3, Q4.2, R14.1; no longer MOTOR_PWR.PIN2, MOTOR_PWR.PIN2-LEAD, Q3.D, Q4.S, R8.1
- net SC: now also MOTOR_PWR1.PIN1, Q1.3, Q2.2; no longer MOTOR_PWR.PIN1, MOTOR_PWR.PIN1-LEAD, Q1.D, Q2.S
- net SI_CAM1: now also CAMERA1.4; no longer CAMERA1.3
- net SI_CAM2: now also CAMERA2.4; no longer CAMERA2.3
- net VBB: now also CONN1.PIN2, MOTOR_PWR.PIN2, Q2.3, Q4.3, Q6.3, U$5.+; no longer Q2.D, Q4.D, Q6.D, U$1.+
- net VDD: now also 3.3V_REGULATOR.IN, 31.1, C26.+, C27.+, CONN2.PIN2, CONN3.PIN2, HALL_SENSOR.6, L1.P$2, MCU_PWR.2, R20.2, R34.1, R35.1, SERVO.2; no longer 3.3V_REGULATOR.2, 32.1, PWR_OUT.2, R17.1, R18.1
Routing:
- net 5V_SERVO: track 159.7 -> 0.00 mm, vias 1 -> 0
- net VBB: track 94.4 -> 242.8 mm, vias 2 -> 0
- net VDD: track 142.4 -> 269.5 mm, vias 3 -> 0
- net GND: track 136.5 -> 253.3 mm, vias 17 -> 14
- net N$2: track 90.5 -> 0.00 mm, vias 4 -> 0
- net PTB9: track 85.5 -> 0.00 mm
- net PTA1: track 78.4 -> 0.00 mm
- net HA: track 183.1 -> 110.7 mm, vias 2 -> 0
- net SELECT: track 0.00 -> 72.3 mm
- net PTA2: track 69.5 -> 0.00 mm
- net UP: track 0.00 -> 62.9 mm
- net SB: track 47.3 -> 107.9 mm
- net DOWN: track 0.00 -> 57.5 mm
- net N$47: track 0.00 -> 54.3 mm, vias 0 -> 2
- net SA: track 50.8 -> 105.0 mm, vias 2 -> 0
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- added copper zone on layer 1, net 3.3V
- added copper zone on layer 1, net GND
Other:
- board size 216.8 x 88.9 mm -> 125.7 x 231.1 mm
- board text removed: "EE192 Team 1"
