File: EE192_Sp17_Team01_combo.sch (EAGLE design)
At the start: 90 parts, among them J1 FRDM-K64F, Q1 IRFS3006PBF, Q2 IRFS3006PBF, Q3 IRFS3006PBF, Q4 IRFS3006PBF, Q5 IRFS3006PBF, Q6 IRFS3006PBF, Q7 IRFS3006PBF

Commit message: Add rev 2 boards
Add rev 2 boards, update to MCU and power circuitry
Parts:
- removed C7: (no value), rcl:C-USC0805
- removed PWR_OUT: (no value), ee192TomasVersion:M031X03-MTA
- removed U$1: TAMIYA, ee192TomasVersion:TAMIYA
- added C13: (no value), rcl:C-USC0805
- added CONN1, CONN2, CONN3: ANDERSON_PP_DOUBLEVERTICAL, ee192:ANDERSON_PP_DOUBLEVERTICAL
- added LED1: (no value), led:LEDCHIPLED_0805
- added MCU_PWR: (no value), ee192:M031X03-MTA
- added MOTOR_PWR1: ANDERSON_PP_TRIPVERT, ee192:ANDERSON_PP_TRIPVERT
- added R34, R35: 50kohm, rcl:R-US_R0805
- added SV1, SV2, SV3, SV4: (no value), con-lstb:MA08-2
- added U$5: TAMIYA, ee192:TAMIYA
- 3.3V_REGULATOR: device v-reg:LM138-TL -> v-reg:78MXXL
- D1: value BAT60J -> 1N5908; device diode:BAT60J -> diode:1N5908
- MOTOR_PWR: value ANDERSON_PP_TRIPHORIZ -> ANDERSON_PP_DOUBLEVERTICAL; device ee192:ANDERSON_PP_TRIPHORIZ -> ee192:ANDERSON_PP_DOUBLEVERTICAL
- Q1, Q2, Q3, Q4, Q5, Q6: value IRFS3006PBF -> (none); device ee192TomasVersion:IRFS3006PBF -> ee192:IRFS3006PBFTO263PACKAGE
- R1, R2: value 50ohm -> (none); device rcl:R-US_R0805 -> resistor:R-US_R0805
- R11, R7: value 10kohm -> 50ohm
- R13, R14: value 50kohm -> 10kohm
Connections:
- removed net 5V_SERVO: 3.3V_REGULATOR.IN, 31.1, C26.+, C27.+, HALL_SENSOR.6, L1.P$2, PWR_OUT.1, R20.2, SERVO.2
- removed net N$35 (its old number): Q4.G, R2.2, R8.2
- removed net PTA1: J1.PTA1, UP.2.1
- removed net PTA2: DOWN.2.1, J1.PTA2
- removed net PTB9: J1.PTB9, SELECT.2.1
- new net 3V3: 3.3V_REGULATOR.OUT, 32.1, MCU_PWR.1
- new net CONN_15_16: SV4.16, SV4.2
- new net DOWN: DOWN.2.1, J1.PTD3
- new net HA_OUT: J1.PTB11, R1.2, R2.2
- new net N$13: SV2.10, SV2.12, SV2.14, SV2.16, SV2.2, SV2.4, SV2.6, SV2.8
- new net N$38: Q6.G, R4.2, R8.1
- new net N$39: Q2.G, R6.2, R9.2
- new net N$46: Q4.G, R14.2, R3.2
- new net N$47: Q5.G, R10.1, R7.2
- new net N$52: Q1.G, R11.2, R12.1
- new net N$53: LED1.C, MOTOR_PREDRIVER.FAULT
- new net N$54: LED1.A, R15.2
- new net N$6: SV3.16, SV3.2
- new net N$7: SV3.1, SV3.15
- new net RST_SCRN: J1.PTD2, SCREEN.3
- new net SELECT: J1.PTC4, SELECT.2.1
- new net UP: J1.PTD0, UP.2.1
- net 3.3V: now also CAMERA1.2, CAMERA2.2
- net 5V: now also SCREEN.4; no longer CAMERA1.2, CAMERA2.2, SCREEN.1
- net BRAKEN: now also J1.PTB9, R18.1; no longer J1.PTD3, R16.1
- net CELL_A: now also BATT_SENSE.3; no longer BATT_SENSE.2
- net CELL_AB: now also BATT_SENSE.2; no longer BATT_SENSE.3
- net CELL_ABC: now also BATT_SENSE.1; no longer BATT_SENSE.4
- net CLK: now also SCREEN.2; no longer SCREEN.5
- net CLK_CAM1: now also CAMERA1.3; no longer CAMERA1.4
- net CLK_CAM2: now also CAMERA2.3; no longer CAMERA2.4
- net DATA: now also SCREEN.1; no longer SCREEN.4
- net DIR: now also R17.1; no longer R14.1
- net ENABLE: now also R16.1; no longer R13.1
- net GHA: now also R4.1; no longer R1.1
- net GHB: now also R3.1; no longer R2.1
- net GHC: now also R6.1; no longer R3.1
- net GLA: now also R7.1; no longer R4.1
- net GLC: now also R11.1; no longer R6.1
- net GND: now also 3.3V_REGULATOR.GND, BATT_SENSE.4, C13.2, CONN1.GND, CONN2.GND, CONN3.GND, MCU_PWR.3, MOTOR_PWR.GND, R17.2, R18.2, R2.1, SCREEN.5, U$5.-; no longer 3.3V_REGULATOR.ADJ, BATT_SENSE.1, C7.2, PWR_OUT.3, R11.2, R14.2, SCREEN.2, U$1.-
- net HA: now also HALL_MCU.3, R1.1, R35.2; no longer HALL_MCU.1, J1.PTD0, R19.2
- net HB: now also J1.PTA2, R34.2; no longer R18.2
- net HC: now also HALL_MCU.1, R19.2; no longer HALL_MCU.3, R17.2
- net MEAS_CELL_A: now also BATT_SENSE1.4; no longer BATT_SENSE1.2, BMS.4
- net MEAS_CELL_C: now also BATT_SENSE1.2, BMS.4; no longer BATT_SENSE1.4
- net N$10: now also SV3.14; no longer Q1.G, R12.1, R6.2
- net N$2: now also SV2.1, SV2.11, SV2.13, SV2.15, SV2.3, SV2.5, SV2.7, SV2.9; no longer Q3.G, R11.1, R5.2
- net N$22: now also SV1.10, SV1.12, SV1.14, SV1.16, SV1.2, SV1.4, SV1.6, SV1.8; no longer Q6.G, R1.2, R7.1
- net N$26: now also SV1.1, SV1.11, SV1.13, SV1.15, SV1.3, SV1.5, SV1.7, SV1.9; no longer Q5.G, R10.1, R4.2
- net N$32: now also SV4.1, SV4.15; no longer Q2.G, R3.2, R9.2
- net N$40: now also Q3.G, R13.1, R5.2; no longer J1.PTB11
- net N$5: no longer MOTOR_PREDRIVER.FAULT, R15.2
- net PWM_SERVO: now also J1.PTA1; no longer J1.PTD2
- net RST: no longer J1.PTC4, SCREEN.3
- net SA: now also C13.1, MOTOR_PWR1.P$3, R8.2; no longer C7.1, MOTOR_PWR.P$3, R7.2
- net SB: now also MOTOR_PWR1.P$2, R14.1; no longer MOTOR_PWR.P$2, R8.1
- net SC: now also MOTOR_PWR1.P$1; no longer MOTOR_PWR.P$1
- net SI_CAM1: now also CAMERA1.4; no longer CAMERA1.3
- net SI_CAM2: now also CAMERA2.4; no longer CAMERA2.3
- net VBB: now also CONN1.VCC, MOTOR_PWR.VCC, U$5.+; no longer U$1.+
- net VDD: now also 3.3V_REGULATOR.IN, 31.1, C26.+, C27.+, CONN2.VCC, CONN3.VCC, HALL_SENSOR.6, L1.P$2, MCU_PWR.2, R20.2, R34.1, R35.1, SERVO.2; no longer 3.3V_REGULATOR.OUT, 32.1, PWR_OUT.2, R17.1, R18.1
Other:
- note added: "Voltage Divider"
